File: Repo - Eletronica/Esquemáticos/Segundo esquemático/Segundo esquemático.kicad_sch (KiCad schematic)
At the start: 27 parts, among them M1 Motor Esquerdo, M2 Motor Direito, Q1 BC547, Q2 BC547, SW1 Chave/Interruptor, SW2 Chave/Interruptor, U2 Medidor de Corrente ACS712, U3 Sensor 1 TCRT500, U4 Sensor 2 TCRT500, U5 Sensor 3 TCRT500, U6 Sensor 4 TCRT500

Commit message: Att
Novas atualizações no esquemático
Parts:
- added R10, R11, R12, R9: 1000, symbol Device:R
- R1, R2, R3, R4, R7, R8: value 500 -> 560
Connections:
- net +5V: now also U3.COLL, U4.COLL, U5.COLL, U6.COLL
- net Earth: now also A1.6 (GND), R10.1, R11.1, R12.1, R9.1; no longer A1.29 (GND), U3.E, U4.E, U5.E, U6.E
- net at A1.11 (A2): now also U4.E, R10.2; no longer U4.COLL
- net at A1.10 (A1): now also U3.E, R9.2; no longer U3.COLL
- net at A1.12 (A3): now also U5.E, R11.2; no longer U5.COLL
- net at A1.13 (SDA/A4): now also U6.E, R12.2; no longer U6.COLL
- new net: U2.8 (VCC), U8. (Vcc), U9. (Vcc)
Other:
- note added: "2 de Maio de 2024"
- note removed: "18 de Abril de 2024"

Commit message: Atualização
Atualizei as informações para o segundo ponto de controle
Connections:
- new net: U2.8 (VCC), U8. (Vcc), U9. (Vcc)
Other:
- note removed: "2 de Maio de 2024"
- note removed: "Terceiro Esquemático do Circuito do Robô"
- company: (none) -> Universidade de Brasília 
- title: (none) -> Projeto K.A.T.I.A.U
Changed lines of the file:
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@@
 (kicad_sch (version 20230121) (generator eeschema)
   (paper "A4")
+  (title_block
+    (title "Projeto K.A.T.I.A.U")
+    (date "2024-05-13")
+    (rev "Pedro Zago")
+    (company "Universidade de Brasília ")
+    (comment 1 "Grupo 2")
+    (comment 2 "Projeto Integrador de Engenharia 1 ")
+  )
   (junction (at 151.13 40.64) (diameter 0) (color 0 0 0 0)
   )
@@
     (stroke (width 0) (type default))
   )
-  (wire (pts (xy 198.12 86.36) (xy 196.85 85.09))
-    (stroke (width 0) (type default))
-  )
-  (wire (pts (xy 74.93 64.77) (xy 86.36 64.77))
-    (stroke (width 0) (type default))
-  )
   (wire (pts (xy 236.22 138.43) (xy 236.22 142.24))
     (stroke (width 0) (type default))
@@
     (stroke (width 0) (type default))
   )
+  (wire (pts (xy 74.93 67.31) (xy 92.71 67.31))
+    (stroke (width 0) (type default))
+  )
   (wire (pts (xy 144.78 22.86) (xy 144.78 31.75))
     (stroke (width 0) (type default))
@@
     (stroke (width 0) (type default))
   )
-  (wire (pts (xy 92.71 73.66) (xy 86.36 67.31))
-    (stroke (width 0) (type default))
-  )
   (wire (pts (xy 227.33 99.06) (xy 229.87 99.06))
     (stroke (width 0) (type default))
   )
+  (wire (pts (xy 228.6 29.21) (xy 228.6 35.56))
+    (stroke (width 0) (type default))
+  )
   (wire (pts (xy 107.95 55.88) (xy 115.57 55.88))
     (stroke (width 0) (type default))
@@
     (stroke (width 0) (type default))
   )
+  (wire (pts (xy 109.22 114.3) (xy 109.22 119.38))
+    (stroke (width 0) (type default))
+  )
   (wire (pts (xy 82.55 114.3) (xy 82.55 121.92))
     (stroke (width 0) (type default))
@@
     (stroke (width 0) (type default))
   )
+  (wire (pts (xy 99.06 64.77) (xy 99.06 74.93))
+    (stroke (width 0) (type default))
+  )
   (wire (pts (xy 115.57 40.64) (xy 132.08 40.64))
     (stroke (width 0) (type default))
@@
     (stroke (width 0) (type default))
   )
-  (wire (pts (xy 196.85 29.21) (xy 222.25 29.21))
+  (wire (pts (xy 196.85 29.21) (xy 228.6 29.21))
     (stroke (width 0) (type default))
   )
@@
     (stroke (width 0) (type default))
   )
-  (wire (pts (xy 74.93 62.23) (xy 101.6 62.23))
-    (stroke (width 0) (type default))
-  )
   (wire (pts (xy 87.63 173.99) (xy 87.63 177.8))
     (stroke (width 0) (type default))
@@
     (stroke (width 0) (type default))
   )
-  (wire (pts (xy 88.9 67.31) (xy 91.44 67.31))
-    (stroke (width 0) (type default))
-  )
   (wire (pts (xy 144.78 48.26) (xy 144.78 67.31))
     (stroke (width 0) (type default))
@@
     (stroke (width 0) (type default))
   )
-  (wire (pts (xy 92.71 73.66) (xy 92.71 92.71))
+  (wire (pts (xy 92.71 67.31) (xy 92.71 92.71))
     (stroke (width 0) (type default))
   )
@@
     (stroke (width 0) (type default))
   )
-  (wire (pts (xy 74.93 67.31) (xy 86.36 67.31))
-    (stroke (width 0) (type default))
-  )
-  (wire (pts (xy 101.6 62.23) (xy 107.95 55.88))
-    (stroke (width 0) (type default))
-  )
   (wire (pts (xy 74.93 59.69) (xy 96.52 59.69))
     (stroke (width 0) (type default))
@@
     (stroke (width 0) (type default))
   )
-  (wire (pts (xy 91.44 67.31) (xy 99.06 74.93))
+  (wire (pts (xy 109.22 119.38) (xy 115.57 119.38))
     (stroke (width 0) (type default))
   )
@@
     (stroke (width 0) (type default))
   )
-  (wire (pts (xy 147.32 29.21) (xy 144.78 31.75))
-    (stroke (width 0) (type default))
-  )
   (wire (pts (xy 151.13 59.69) (xy 151.13 62.23))
     (stroke (width 0) (type default))
   )
-  (wire (pts (xy 96.52 59.69) (xy 96.52 48.26))
+  (wire (pts (xy 96.52 39.37) (xy 96.52 59.69))
     (stroke (width 0) (type default))
   )
@@
     (stroke (width 0) (type default))
   )
+  (wire (pts (xy 74.93 64.77) (xy 99.06 64.77))
+    (stroke (width 0) (type default))
+  )
   (wire (pts (xy 130.81 91.44) (xy 151.13 91.44))
     (stroke (width 0) (type default))
@@
     (stroke (width 0) (type default))
   )
+  (wire (pts (xy 74.93 62.23) (xy 107.95 62.23))
+    (stroke (width 0) (type default))
+  )
   (wire (pts (xy 115.57 55.88) (xy 115.57 59.69))
     (stroke (width 0) (type default))
@@
     (stroke (width 0) (type default))
   )
-  (wire (pts (xy 109.22 114.3) (xy 115.57 119.38))
-    (stroke (width 0) (type default))
-  )
   (wire (pts (xy 110.49 48.26) (xy 115.57 48.26))
     (stroke (width 0) (type default))
@@
     (stroke (width 0) (type default))
   )
+  (wire (pts (xy 196.85 85.09) (xy 198.12 85.09))
+    (stroke (width 0) (type default))
+  )
   (wire (pts (xy 115.57 74.93) (xy 115.57 78.74))
     (stroke (width 0) (type default))
@@
     (stroke (width 0) (type default))
   )
+  (wire (pts (xy 107.95 55.88) (xy 107.95 62.23))
+    (stroke (width 0) (type default))
+  )
   (wire (pts (xy 236.22 115.57) (xy 237.49 115.57))
     (stroke (width 0) (type default))
@@
     (stroke (width 0) (type default))
   )
-  (wire (pts (xy 105.41 39.37) (xy 115.57 39.37))
-    (stroke (width 0) (type default))
-  )
-  (wire (pts (xy 198.12 86.36) (xy 198.12 104.14))
+  (wire (pts (xy 96.52 39.37) (xy 115.57 39.37))
+    (stroke (width 0) (type default))
+  )
+  (wire (pts (xy 198.12 85.09) (xy 198.12 104.14))
     (stroke (width 0) (type default))
   )
@@
     (stroke (width 0) (type default))
   )
-  (wire (pts (xy 88.9 67.31) (xy 86.36 64.77))
-    (stroke (width 0) (type default))
-  )
   (wire (pts (xy 194.31 41.91) (xy 219.71 41.91))
     (stroke (width 0) (type default))
   )
+  (wire (pts (xy 147.32 29.21) (xy 147.32 31.75))
+    (stroke (width 0) (type default))
+  )
   (wire (pts (xy 243.84 90.17) (xy 243.84 93.98))
     (stroke (width 0) (type default))
   )
+  (wire (pts (xy 144.78 31.75) (xy 147.32 31.75))
+    (stroke (width 0) (type default))
+  )
   (wire (pts (xy 130.81 48.26) (xy 133.35 48.26))
     (stroke (width 0) (type default))
   )
-  (wire (pts (xy 96.52 48.26) (xy 105.41 39.37))
-    (stroke (width 0) (type default))
-  )
   (wire (pts (xy 130.81 36.83) (xy 151.13 36.83))
     (stroke (width 0) (type default))
@@
     (stroke (width 0) (type default))
   )
-  (wire (pts (xy 222.25 29.21) (xy 228.6 35.56))
-    (stroke (width 0) (type default))
-  )
   (wire (pts (xy 237.49 81.28) (xy 238.76 81.28))
     (stroke (width 0) (type default))
@@
   (text "Medição" (at 30.48 156.21 0)
     (effects (font (size 1.27 1.27) (color 0 0 0 1)) (justify left bottom))
-  )
-  (text "2 de Maio de 2024\n" (at 207.01 194.31 0)
-    (effects (font (size 1.27 1.27) bold) (justify left bottom))
   )
   (text "Encoder M1" (at 50.8 135.89 0)
@@
     (effects (font (size 1.27 1.27) (color 0 0 0 1)) (justify left bottom))
   )
-  (text "Terceiro Esquemático do Circuito do Robô" (at 186.69 190.5 0)
-    (effects (font (size 1.27 1.27) (thickness 0.254) bold) (justify left bottom))
-  )
   (text "Encoder M2\n" (at 83.82 135.89 0)
